Commit message: Updated urdf file with xacro

File: models/lidar_robot_v1.urdf (robot description, URDF)
Before this commit: robot twd_lidar_robot, 9 links, 8 joints
Links:
- link base_link: geometry collision box size=${base_length} ${base_width} ${base_height}; visual mesh filename=package://twd_lidar_robot/meshes/robot_base_link.dae
- link left_wheel: geometry collision cylinder length=${wheel_width} radius=${wheel_radius}; visual mesh filename=package://twd_lidar_robot/meshes/left_wheel.dae
- link right_wheel: geometry collision cylinder length=${wheel_width} radius=${wheel_radius}; visual mesh filename=package://twd_lidar_robot/meshes/right_wheel.dae
- link rplidar_top: mass 0.07 -> None
Joints:
- joint base_joint: origin xyz=0 0 0.045 rpy=0 0 0 -> xyz=0 0 ${(wheel_radius+wheel_zoff)} rpy=0 0 0
- joint left_wheel_hinge: origin xyz=-0.028 0.0675 -0.0125 rpy=0 0 0 -> xyz=-0.028 0.0675 -${wheel_zoff} rpy=0 0 0
- joint right_wheel_hinge: origin xyz=-0.028 -0.075 -0.0125 rpy=0 0 0 -> xyz=-0.028 -0.075 -${wheel_zoff} rpy=0 0 0

Commit message: Successfully implemented SLAM using lidar robot

File: models/lidar_robot_v1.urdf (robot description, URDF)
Before this commit: robot twd_lidar_robot, 9 links, 8 joints
Links:
- added link imu_link
- link left_wheel: geometry collision cylinder length=${wheel_width} radius=${wheel_outer_radius}; visual mesh filename=package://twd_lidar_robot/meshes/left_wheel.dae
- link right_wheel: geometry collision cylinder length=${wheel_width} radius=${wheel_outer_radius}; visual mesh filename=package://twd_lidar_robot/meshes/right_wheel.dae
Joints:
- added joint imu_joint: type fixed, parent base_link, child imu_link, origin xyz=-0.10 0 0.05 rpy=0 0 0
- joint base_joint: origin xyz=0 0 ${(wheel_radius+wheel_zoff)} rpy=0 0 0 -> xyz=0 0 ${(wheel_outer_radius+wheel_zoff)} rpy=0 0 0
- joint caster_wheel_to_mount: limit lower=-3.1415 upper=3.1415 effort=30 velocity=5.0 -> (none)
